File: hardware/christmastreedriver.kicad_sch (KiCad schematic)
At the start: 2 parts, among them J1 M8S-03PMMR-SF8001, J2 USB4105

Commit message: Flipped some stuff
Connections:
- net Bridge Driver/A: now also J1.3 (Pin_3); no longer J1.1 (Pin_1)
- net Bridge Driver/B: now also J1.1 (Pin_1); no longer J1.3 (Pin_3)
Other:
- sheet Microcontroller ports: added PD_Alert, PD_Attach, PD_Reset; removed none
- sheet USB PD ports: added Alert, Attach; removed none
- moved on the sheet: J1
