File: hardware/microcontroller.kicad_sch (KiCad schematic)
At the start: 29 parts, among them Q2 BC817RAPNZ, SW1 EVQPUC, SW2 EVQPUC, U3 CP2102N-A02-GQFN28R, U4 ESP32-PICO-D4

Commit message: Generated first bom
Parts:
- removed R16, R17: 0, Resistor_SMD:R_0402_1005Metric, symbol frank_partdb:CR0402AJ/-000GLF
- U3: footprint Package_DFN_QFN:QFN-28-1EP_5x5mm_P0.5mm_EP3.35x3.35mm -> Package_DFN_QFN:QFN-28-1EP_5x5mm_P0.5mm_EP3.35x3.35mm_ThermalVias
Connections:
- net Current Sense: now also U4.22 (IO2); no longer U4.35 (IO18)
- net DRIVE_A: now also U4.16 (IO27); no longer U4.10 (IO34)
- net DRIVE_B: now also U4.17 (IO14); no longer U4.11 (IO35)
- net Fault: now also U4.21 (IO15); no longer U4.12 (IO32)
- net USB_D+: now also D1.1 (K1); no longer D1.2 (K2)
- net USB_D-: now also D1.2 (K2); no longer D1.1 (K1)
Other:
- moved on the sheet: D1

Commit message: Flipped some stuff
Connections:
- net GND: no longer AE1.2 (PCB_Trace)
- net PD_Attach: now reaches U4.12 (IO32)
- net PD_Alert: now reaches U4.35 (IO18)
- net PD_Reset: now reaches U4.38 (IO19)
- no-connect marks 19 -> 20
Changed lines of the file:
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@@
+	)
+	(no_connect
+		(at 107.95 29.21)
 	)
 	(no_connect
@@
 		)
 	)
+	(hierarchical_label "PD_Reset"
+		(shape output)
+		(at 208.28 101.6 180)
+		(fields_autoplaced yes)
+		(effects
+			(font
+				(size 1.27 1.27)
+			)
+			(justify right)
+		)
+	)
 	(hierarchical_label "DRIVE_A"
 		(shape output)
@@
 		)
 	)
+	(hierarchical_label "PD_Alert"
+		(shape input)
+		(at 208.28 99.06 180)
+		(fields_autoplaced yes)
+		(effects
+			(font
+				(size 1.27 1.27)
+			)
+			(justify right)
+		)
+	)
 	(hierarchical_label "SPI_MISO"
 		(shape input)
@@
 			)
 			(justify left)
+		)
+	)
+	(hierarchical_label "PD_Attach"
+		(shape input)
+		(at 208.28 119.38 180)
+		(fields_autoplaced yes)
+		(effects
+			(font
+				(size 1.27 1.27)
+			)
+			(justify right)
 		)
 	)
@@
 					(unit 1)
 				)
-			)
-		)
-	)
-	(symbol
-		(lib_id "power:GND")
-		(at 107.95 29.21 0)
-		(mirror y)
-		(unit 1)
-		(exclude_from_sim no)
-		(in_bom yes)
-		(on_board yes)
-		(dnp no)
-		(fields_autoplaced yes)
-		(property "Reference" "#PWR0104"
-			(at 107.95 35.56 0)
-			(effects
-				(font
-					(size 1.27 1.27)
-				)
-				(hide yes)
-			)
-		)
-		(property "Value" "GND"
-			(at 107.95 34.29 0)
-			(effects
-				(font
-					(size 1.27 1.27)
-				)
-			)
-		)
-		(property "Footprint" ""
-			(at 107.95 29.21 0)
-			(effects
-				(font
-					(size 1.27 1.27)
-				)
-				(hide yes)
-			)
-		)
-		(property "Datasheet" ""
-			(at 107.95 29.21 0)
-			(effects
-				(font
-					(size 1.27 1.27)
-				)
-				(hide yes)
-			)
-		)
-		(property "Description" "Power symbol creates a global label with name \"GND\" , ground"
-			(at 107.95 29.21 0)
-			(effects
-				(font
-					(size 1.27 1.27)
-				)
-				(hide yes)
-			)
-		)
-		(pin "1"
-		)
-		(instances
-			(project "christmastreedriver"
-				(path "/e5e61a32-0573-464a-9319-78c3ec7b0a35/4b97c7ff-a227-414c-9641-03bffe5fba15"
-					(reference "#PWR0104")
-					(unit 1)
-				)
