File: hardware/usb_pd.kicad_sch (KiCad schematic)
At the start: 11 parts, among them Q1 STL9P3LLH6, U1 STUSB4500QTR

Commit message: Generated first bom
Other:
- moved on the sheet: C11, C12, C13, C17, D2, Q1, R21, R22, R23, R24, U1

Commit message: Flipped some stuff
Connections:
- net Attach: now reaches U1.11 (ATTACH)
- net Alert: now reaches U1.19 (ALERT)
Changed lines of the file:
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@@
+	(wire
+		(pts
+			(xy 123.19 115.57) (xy 132.08 115.57)
+		)
+		(stroke
+			(width 0)
+			(type default)
+		)
+	)
 	(wire
 		(pts
@@
 	(wire
 		(pts
-			(xy 118.11 85.09) (xy 132.08 85.09)
+			(xy 123.19 85.09) (xy 132.08 85.09)
 		)
 		(stroke
@@
 		(pts
 			(xy 125.73 118.11) (xy 125.73 120.65)
+		)
+		(stroke
+			(width 0)
+			(type default)
+		)
+	)
+	(wire
+		(pts
+			(xy 167.64 115.57) (xy 162.56 115.57)
 		)
 		(stroke
@@
 	(hierarchical_label "Reset"
 		(shape input)
-		(at 118.11 85.09 180)
+		(at 123.19 85.09 180)
 		(fields_autoplaced yes)
 		(effects
@@
 		)
 	)
+	(hierarchical_label "Alert"
+		(shape output)
+		(at 123.19 115.57 180)
+		(fields_autoplaced yes)
+		(effects
+			(font
+				(size 1.27 1.27)
+			)
+			(justify right)
+		)
+	)
+	(hierarchical_label "Attach"
+		(shape output)
+		(at 167.64 115.57 0)
+		(fields_autoplaced yes)
+		(effects
+			(font
+				(size 1.27 1.27)
+			)
+			(justify left)
+		)
+	)
